Commit message: Added front wheel

File: task_one/urdf/hola_bot.urdf (robot description, URDF)
Before this commit: robot hola_bot, 2 links, 1 joints
Links:
- added link left_wheel, mass 0.062; collision cylinder length=0.02 radius=.03; visual mesh filename=package://hola_bot/meshes/wheel.STL
- added link right_wheel, mass 0.062; collision cylinder length=0.02 radius=.03; visual mesh filename=package://hola_bot/meshes/wheel.STL
Joints:
- added joint left_joint: type continuous, parent base_link, child left_wheel, origin xyz=0 0.17483 -0.0335 rpy=0 0 0, axis 0 -1 0, limit effort=5 velocity=5
- added joint right_joint: type continuous, parent base_link, child right_wheel, origin xyz=0 0.17483 -0.0335 rpy=0 0 0, axis 0 -1 0, limit effort=5 velocity=5

Commit message: updated launch files according to the tasks

File: task_one/urdf/hola_bot.urdf (robot description, URDF)
Before this commit: robot hola_bot, 4 links, 3 joints
Joints:
- joint left_joint: origin xyz=0 0.17483 -0.0335 rpy=0 0 0 -> xyz=-0.15154 -0.0872575 -0.0335 rpy=0 0 0
- joint right_joint: origin xyz=0 0.17483 -0.0335 rpy=0 0 0 -> xyz=0.15154 -0.0872575 -0.0335 rpy=0 0 0

Commit message: task_one part one done

File: task_one/urdf/hola_bot.urdf (robot description, URDF)
Before this commit: robot hola_bot, 4 links, 3 joints
Links:
- link base_link: geometry collision cylinder length=0.005 radius=0.15; visual mesh filename=package://task_one/meshes/base_link.STL
- link front_wheel: geometry collision cylinder length=0.02 radius=.03; visual mesh filename=package://task_one/meshes/wheel.STL
- link left_wheel: geometry collision cylinder length=0.02 radius=.03; visual mesh filename=package://task_one/meshes/wheel.STL
- link right_wheel: geometry collision cylinder length=0.02 radius=.03; visual mesh filename=package://task_one/meshes/wheel.STL
Joints:
- joint left_joint: origin xyz=-0.15154 -0.0872575 -0.0335 rpy=0 0 0 -> xyz=-0.15154 -0.0872575 -0.0335 rpy=0 0 -1.0467
- joint right_joint: origin xyz=0.15154 -0.0872575 -0.0335 rpy=0 0 0 -> xyz=0.15154 -0.0872575 -0.0335 rpy=0 0 1.0467

Commit message: updated urdf according to the instructions

File: task_one/urdf/hola_bot.urdf (robot description, URDF)
Before this commit: robot hola_bot, 4 links, 3 joints
Joints:
- joint left_joint: origin xyz=-0.15154 -0.0872575 -0.0335 rpy=0 0 -1.0467 -> xyz=-0.151407221 -0.087415 -0.0335 rpy=3.14 0 -1.0467
- joint right_joint: origin xyz=0.15154 -0.0872575 -0.0335 rpy=0 0 1.0467 -> xyz=0.151407221 -0.087415 -0.0335 rpy=3.14 0 1.0467
