Commit message: modified urdf visually

File: task_two/urdf/hola_bot.urdf (robot description, URDF)
Before this commit: robot hola_bot, 4 links, 3 joints
Links:
- link base_link: geometry collision cylinder length=0.005 radius=0.15; visual mesh filename=package://task_two/meshes/base_link.obj
- link front_wheel: geometry collision cylinder length=0.02 radius=.03; visual mesh filename=package://task_two/meshes/wheel.STL
- link left_wheel: geometry collision cylinder length=0.02 radius=.03; visual mesh filename=package://task_two/meshes/wheel.STL
- link right_wheel: geometry collision cylinder length=0.02 radius=.03; visual mesh filename=package://task_two/meshes/wheel.STL
